File: pcb/android_header.kicad_sch (KiCad schematic)
At the start: 19 parts, among them J16 Conn_01x03_Pin, J18 Conn_02x20_Counter_Clockwise, Q14 PMOS, Q15 NMOS, U18 CPDV5-5V0U, U21 SN74LVC8T245, U22 SN74LVC8T245

Commit message: Add the last few mystery components to the schematic, update the licence and start on RHSP
Changed lines of the file:
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@@
 		)
 	)
-	(text_box "Pin 6 on the header and the source of Q15 seems to be left floating at about 0.9V. Because the gate is only 1.8V it doesn't turn Q16 on and PJ6 (an input) is never be pulled down even when OE goes low. Am I missing a ground connection here?"
+	(text_box "Pin 6 on the header and the source of Q15 seems to be left floating at about 0.9V. Because the gate is only 1.8V it doesn't turn Q15 on and PJ6 (an input) is never be pulled down even when OE goes low. Am I missing a ground connection here?"
 		(exclude_from_sim no)
 		(at 231.14 137.16 0)
