File: pcb/12v.kicad_sch (KiCad schematic)
At the start: 14 parts, among them J21 Conn_01x02_Socket, J26 Conn_01x02_Pin, Q29 NMOS, U25 Conn_02x03_Counter_Clockwise

Commit message: Add the last few mystery components to the schematic, update the licence and start on RHSP
Parts:
- removed U25: Conn_02x03_Counter_Clockwise, symbol Connector_Generic:Conn_02x03_Counter_Clockwise
- added U25: ZXCT1010, Package_TO_SOT_SMD:SOT-23-5, symbol Amplifier_Current:ZXCT1010
- D5: footprint (none) -> Diode_SMD:D_SOD-882; symbol Device:D -> Diode:PESD5V0S1UL
Connections:
- net GND: now also U25.2 (GND)
- net at R128.2: now also U25.5 (Vs-)
- net at R128.3: now also U25.4 (Vs+)
- net at R124.2, R126?.1: now also U25.3 (OUT)
- no-connect marks 2 -> 0
Other:
- note removed: "Represents a SOT 25 or SOT 23-5 ic that is unidentifed"
- moved on the sheet: C75, R124, R126?

Commit message: Before tear out
Parts:
- R128: value R_Shunt -> 0.003
Changed lines of the file:
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@@
 			)
 		)
-		(property "Value" "R_Shunt"
+		(property "Value" "0.003"
 			(at 160.02 105.41 90)
 			(effects
