File: pcb/5v.kicad_sch (KiCad schematic)
At the start: 13 parts, among them J20 Conn_01x24_Pin, Q19 NMOS, Q20 PMOS, U26 CPDV5-5V0U

Commit message: Before tear out
Changed lines of the file:
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@@
 	(wire
 		(pts
-			(xy 162.56 27.94) (xy 163.83 27.94)
+			(xy 161.29 27.94) (xy 163.83 27.94)
 		)
 		(stroke
@@
 	(global_label "PM2"
 		(shape input)
-		(at 162.56 27.94 180)
+		(at 161.29 27.94 180)
 		(fields_autoplaced yes)
 		(effects
@@
 		)
 		(property "Intersheetrefs" "${INTERSHEET_REFS}"
-			(at 155.6439 27.94 0)
+			(at 154.3739 27.94 0)
 			(effects
 				(font
