File: pcb/vrefa_plus.kicad_sch (KiCad schematic)
At the start: 11 parts

Commit message: Add the last few mystery components to the schematic, update the licence and start on RHSP
Parts:
- removed J? (x3): Conn_01x01_Pin, symbol Connector:Conn_01x01_Pin
- added U17: TL431ASA, Package_TO_SOT_SMD:SOT-23, symbol Reference_Voltage:TL431DBZ
Connections:
- net GND: now also U17.3 (A)
- net VREFA+: now also U17.1 (K)
- net at R74.1, R78?.1: now also U17.2 (REF)
Other:
- note removed: "This is U17. Couldn't find what it is and couldn't find a good way to indicate a generic three pin chip"

Commit message: Before tear out
Connections:
- net GND: now also R74.1; no longer R74.2
- net VREFA+: now also R78?.1; no longer R78?.2
- new net: R74.2, R78?.2, U17.2 (REF)
Other:
- moved on the sheet: C37, C38, C41, C42, R74, R78?, R79?, R80, U17
